Commit message: feat(onrobot_macro): declare mimic joints and velocity state for gz_ros2_control
Co-Authored-By: Claude Opus 5 <noreply@anthropic.com>

File: urdf/onrobot_macro.xacro (robot description, xacro)
@@ -53,5 +53,27 @@
                 <command_interface name="position"/>
                 <state_interface name="position"/>
+                <xacro:if value="${sim_gazebo}">
+                    <!-- GripperActionController claims position + velocity state -->
+                    <state_interface name="velocity"/>
+                </xacro:if>
             </joint>
+            <!-- gz_ros2_control drives mimic joints itself: each must be listed in the same
+                 ros2_control block with the mimicked joint and a multiplier (no offset support,
+                 see finger_joint_multiplier in the rgX_macro.xacro). -->
+            <xacro:if value="${sim_gazebo}">
+                <xacro:macro name="gz_mimic_joint" params="name k">
+                    <joint name="${prefix}${name}">
+                        <param name="mimic">${prefix}finger_width</param>
+                        <param name="multiplier">${k * finger_joint_multiplier}</param>
+                        <state_interface name="position"/>
+                    </joint>
+                </xacro:macro>
+                <xacro:gz_mimic_joint name="finger_joint" k="1"/>
+                <xacro:gz_mimic_joint name="left_inner_knuckle_joint" k="-1"/>
+                <xacro:gz_mimic_joint name="left_inner_finger_joint" k="1"/>
+                <xacro:gz_mimic_joint name="right_outer_knuckle_joint" k="-1"/>
+                <xacro:gz_mimic_joint name="right_inner_knuckle_joint" k="-1"/>
+                <xacro:gz_mimic_joint name="right_inner_finger_joint" k="1"/>
+            </xacro:if>
         </ros2_control>
     </xacro:macro>

Commit message: fix(onrobot_macro): actuate finger_joint instead of massless finger_width in gazebo
Co-Authored-By: Claude Opus 5 <noreply@anthropic.com>

File: urdf/onrobot_macro.xacro (robot description, xacro)
@@ -14,11 +14,14 @@
         port:=502
         ">
+        <!-- In Gazebo the knuckle (finger_joint, [rad]) is actuated instead of the massless
+             finger_width slider ([m]); see onrobot_rgX in rgX_macro.xacro. -->
+        <xacro:property name="actuated_joint" value="${'finger_joint' if sim_gazebo else 'finger_width'}"/>
         <xacro:if value="${onrobot_type == 'rg2'}">
             <xacro:include filename="$(find onrobot_description)/urdf/rg2_macro.xacro"/>
-            <xacro:onrobot_rg2 prefix="${prefix}"/>
+            <xacro:onrobot_rg2 prefix="${prefix}" actuated_joint="${actuated_joint}"/>
         </xacro:if>
         <xacro:if value="${onrobot_type == 'rg6'}">
             <xacro:include filename="$(find onrobot_description)/urdf/rg6_macro.xacro"/>
-            <xacro:onrobot_rg6 prefix="${prefix}"/>
+            <xacro:onrobot_rg6 prefix="${prefix}" actuated_joint="${actuated_joint}"/>
         </xacro:if>
         <!-- Enable the Gazebo Sim (Fortress) ros2_control plugin for simulation.
@@ -50,5 +53,5 @@
                 </xacro:unless>
             </hardware>
-            <joint name="${prefix}finger_width">
+            <joint name="${prefix}${actuated_joint}">
                 <command_interface name="position"/>
                 <state_interface name="position"/>
@@ -59,15 +62,15 @@
             </joint>
             <!-- gz_ros2_control drives mimic joints itself: each must be listed in the same
-                 ros2_control block with the mimicked joint and a multiplier (no offset support,
-                 see finger_joint_multiplier in the rgX_macro.xacro). -->
+                 ros2_control block with the mimicked joint and a multiplier (no offset support).
+                 finger_width is left out on purpose: it has no mass or collision, so nothing
+                 physical depends on it, and robot_state_publisher derives it from the URDF. -->
             <xacro:if value="${sim_gazebo}">
                 <xacro:macro name="gz_mimic_joint" params="name k">
                     <joint name="${prefix}${name}">
-                        <param name="mimic">${prefix}finger_width</param>
-                        <param name="multiplier">${k * finger_joint_multiplier}</param>
+                        <param name="mimic">${prefix}finger_joint</param>
+                        <param name="multiplier">${k}</param>
                         <state_interface name="position"/>
                     </joint>
                 </xacro:macro>
-                <xacro:gz_mimic_joint name="finger_joint" k="1"/>
                 <xacro:gz_mimic_joint name="left_inner_knuckle_joint" k="-1"/>
                 <xacro:gz_mimic_joint name="left_inner_finger_joint" k="1"/>
