Commit message: fix(rg_macros): move gripper_tcp inside macro so it can be instantiated twice
Co-Authored-By: Claude Opus 5 <noreply@anthropic.com>

File: urdf/rg2_macro.xacro (robot description, xacro)
@@ -59,10 +59,4 @@
     <xacro:finger_joints prefix="${prefix}" fingerprefix="right" reflect="-1.0"/>
   </xacro:macro>
-  <link name="${prefix}gripper_tcp" />
-  <joint name="${prefix}tcp_joint" type="fixed">
-    <origin xyz="0 0 0.218" rpy="0 0 0" />
-    <parent link="${prefix}onrobot_base_link" />
-    <child link="${prefix}gripper_tcp" />
-  </joint>
   <xacro:macro name="onrobot_rg2" params="prefix">
     <xacro:onrobot_base_link prefix="${prefix}" />
@@ -72,4 +66,10 @@
     <xacro:right_outer_knuckle_joint prefix="${prefix}"/>
     <xacro:transmission_macro prefix="${prefix}" joint_name="finger_width"/>
+    <link name="${prefix}gripper_tcp" />
+    <joint name="${prefix}tcp_joint" type="fixed">
+      <origin xyz="0 0 0.218" rpy="0 0 0" />
+      <parent link="${prefix}onrobot_base_link" />
+      <child link="${prefix}gripper_tcp" />
+    </joint>
   </xacro:macro>
 </robot>

File: urdf/rg6_macro.xacro (robot description, xacro)
@@ -59,10 +59,4 @@
     <xacro:finger_joints prefix="${prefix}" fingerprefix="right" reflect="-1.0"/>
   </xacro:macro>
-  <link name="${prefix}gripper_tcp"/>
-  <joint name="${prefix}tcp_joint" type="fixed">
-    <origin xyz="0 0 0.268" rpy="0 0 0" />
-    <parent link="${prefix}onrobot_base_link" />
-    <child link="${prefix}gripper_tcp" />
-  </joint>
   <xacro:macro name="onrobot_rg6" params="prefix">
     <xacro:onrobot_base_link prefix="${prefix}" />
@@ -72,4 +66,10 @@
     <xacro:right_outer_knuckle_joint prefix="${prefix}"/>
     <xacro:transmission_macro prefix="${prefix}" joint_name="finger_width"/>
+    <link name="${prefix}gripper_tcp"/>
+    <joint name="${prefix}tcp_joint" type="fixed">
+      <origin xyz="0 0 0.268" rpy="0 0 0" />
+      <parent link="${prefix}onrobot_base_link" />
+      <child link="${prefix}gripper_tcp" />
+    </joint>
   </xacro:macro>
 </robot>

Commit message: fix(rg_macros): remove finger joint mimic offsets and give finger_width_mock_link inertia for gazebo
Co-Authored-By: Claude Opus 5 <noreply@anthropic.com>

File: urdf/rg2_macro.xacro (robot description, xacro)
@@ -2,12 +2,20 @@
 <robot xmlns:xacro="http://ros.org/wiki/xacro">
   <xacro:property name="onrobot_type" value="rg2" />
+  <!--
+    finger_joint = finger_joint_multiplier * finger_width, with NO offset.
+    gz_ros2_control mimic joints support a multiplier only, so each finger joint's zero is placed
+    at finger_width = 0 by rotating its joint origin by the former offset about the joint axis and
+    shifting its limits by the same amount. Link poses for a given finger_width are unchanged.
+  -->
+  <xacro:property name="finger_joint_offset" value="0.785398" />
+  <xacro:property name="finger_joint_multiplier" value="${0.85 * ((-0.558505 - 0.785398) / 0.110)}" />
   <xacro:include filename="$(find onrobot_description)/urdf/inc/rg_common.xacro" />
   <xacro:macro name="inner_knuckle_joint" params="prefix fingerprefix reflect">
     <joint name="${prefix}${fingerprefix}_inner_knuckle_joint" type="revolute">
-      <origin xyz="0 ${reflect * -0.007678} 0.1422970" rpy="0 0 ${(reflect - 1) * pi / 2}" />
+      <origin xyz="0 ${reflect * -0.007678} 0.1422970" rpy="${-finger_joint_offset} 0 ${(reflect - 1) * pi / 2}" />
       <parent link="${prefix}onrobot_base_link" />
       <child link="${prefix}${fingerprefix}_inner_knuckle" />
       <axis xyz="1 0 0" />
-      <limit lower="-0.785398" upper="0.785398" velocity="100.0" effort="1000" />
+      <limit lower="${-0.785398 + finger_joint_offset}" upper="${0.785398 + finger_joint_offset}" velocity="100.0" effort="1000" />
       <mimic joint="${prefix}finger_joint" multiplier="-1" offset="0" />
     </joint>
@@ -15,9 +23,9 @@
   <xacro:macro name="inner_finger_joint" params="prefix fingerprefix">
     <joint name="${prefix}${fingerprefix}_inner_finger_joint" type="revolute">
-      <origin xyz="0 ${-(0.056770-0.017178)} ${0.163974-0.125797}" rpy="0 0 0" />
+      <origin xyz="0 ${-(0.056770-0.017178)} ${0.163974-0.125797}" rpy="${finger_joint_offset} 0 0" />
       <parent link="${prefix}${fingerprefix}_outer_knuckle" />
       <child link="${prefix}${fingerprefix}_inner_finger" />
       <axis xyz="1 0 0" />
-      <limit lower="-0.872665" upper="0.872665" velocity="100.0" effort="1000" />
+      <limit lower="${-0.872665 - finger_joint_offset}" upper="${0.872665 - finger_joint_offset}" velocity="100.0" effort="1000" />
       <mimic joint="${prefix}finger_joint" multiplier="1" offset="0" />
     </joint>
@@ -30,5 +38,11 @@
   </xacro:macro>
   <xacro:macro name="finger_joint" params="prefix">
-    <link name="${prefix}finger_width_mock_link"/>
+    <!-- tiny inertia: without it the URDF->SDF conversion drops this link and finger_width with it -->
+    <link name="${prefix}finger_width_mock_link">
+      <inertial>
+        <mass value="0.001" />
+        <inertia ixx="1e-7" ixy="0" ixz="0" iyy="1e-7" iyz="0" izz="1e-7" />
+      </inertial>
+    </link>
     <joint name="${prefix}finger_width" type="prismatic">
       <origin xyz="0 0 0" rpy="0 0 0" />
@@ -39,10 +53,10 @@
     </joint>
     <joint name="${prefix}finger_joint" type="revolute">
-      <origin xyz="0 -0.017178 0.125797" rpy="0 0 0" />
+      <origin xyz="0 -0.017178 0.125797" rpy="${-finger_joint_offset} 0 0" />
       <parent link="${prefix}onrobot_base_link" />
       <child link="${prefix}left_outer_knuckle" />
       <axis xyz="-1 0 0" />
-      <limit lower="-0.558505" upper="0.785398" velocity="100.0" effort="1000" />
-      <mimic joint="${prefix}finger_width" multiplier="${0.85 * ((-0.558505 - 0.785398) / 0.110)}" offset="0.785398" />
+      <limit lower="${-0.558505 - finger_joint_offset}" upper="${0.785398 - finger_joint_offset}" velocity="100.0" effort="1000" />
+      <mimic joint="${prefix}finger_width" multiplier="${finger_joint_multiplier}" offset="0" />
     </joint>
     <xacro:finger_joints prefix="${prefix}" fingerprefix="left" reflect="1.0"/>
@@ -50,9 +64,9 @@
   <xacro:macro name="right_outer_knuckle_joint" params="prefix">
     <joint name="${prefix}right_outer_knuckle_joint" type="revolute">
-      <origin xyz="0 0.017178 0.125797" rpy="0 0 ${pi}" />
+      <origin xyz="0 0.017178 0.125797" rpy="${-finger_joint_offset} 0 ${pi}" />
       <parent link="${prefix}onrobot_base_link" />
       <child link="${prefix}right_outer_knuckle" />
       <axis xyz="1 0 0" />
-      <limit lower="-0.785398" upper="0.785398" velocity="100.0" effort="1000" />
+      <limit lower="${-0.785398 + finger_joint_offset}" upper="${0.785398 + finger_joint_offset}" velocity="100.0" effort="1000" />
       <mimic joint="${prefix}finger_joint" multiplier="-1" offset="0" />
     </joint>

File: urdf/rg6_macro.xacro (robot description, xacro)
@@ -2,12 +2,20 @@
 <robot xmlns:xacro="http://ros.org/wiki/xacro">
   <xacro:property name="onrobot_type" value="rg6" />
+  <!--
+    finger_joint = finger_joint_multiplier * finger_width, with NO offset.
+    gz_ros2_control mimic joints support a multiplier only, so each finger joint's zero is placed
+    at finger_width = 0 by rotating its joint origin by the former offset about the joint axis and
+    shifting its limits by the same amount. Link poses for a given finger_width are unchanged.
+  -->
+  <xacro:property name="finger_joint_offset" value="0.628319" />
+  <xacro:property name="finger_joint_multiplier" value="${0.88 * ((-0.628319 - 0.628319) / 0.160)}" />
   <xacro:include filename="$(find onrobot_description)/urdf/inc/rg_common.xacro" />
   <xacro:macro name="inner_knuckle_joint" params="prefix fingerprefix reflect">
     <joint name="${prefix}${fingerprefix}_inner_knuckle_joint" type="revolute">
-      <origin xyz="0 ${reflect * -0.012720} 0.159500" rpy="0 0 ${(reflect - 1) * pi / 2}" />
+      <origin xyz="0 ${reflect * -0.012720} 0.159500" rpy="${-finger_joint_offset} 0 ${(reflect - 1) * pi / 2}" />
       <parent link="${prefix}onrobot_base_link" />
       <child link="${prefix}${fingerprefix}_inner_knuckle" />
       <axis xyz="1 0 0" />
-      <limit lower="-0.628319" upper="0.628319" velocity="2.0" effort="1000" />
+      <limit lower="${-0.628319 + finger_joint_offset}" upper="${0.628319 + finger_joint_offset}" velocity="2.0" effort="1000" />
       <mimic joint="${prefix}finger_joint" multiplier="-1" offset="0" />
     </joint>
@@ -15,9 +23,9 @@
   <xacro:macro name="inner_finger_joint" params="prefix fingerprefix">
     <joint name="${prefix}${fingerprefix}_inner_finger_joint" type="revolute">
-      <origin xyz="0 ${-(0.071447-0.024112)} ${0.201308-0.136813}" rpy="0 0 0" />
+      <origin xyz="0 ${-(0.071447-0.024112)} ${0.201308-0.136813}" rpy="${finger_joint_offset} 0 0" />
       <parent link="${prefix}${fingerprefix}_outer_knuckle" />
       <child link="${prefix}${fingerprefix}_inner_finger" />
       <axis xyz="1 0 0" />
-      <limit lower="-0.872665" upper="0.872665" velocity="2.0" effort="1000" />
+      <limit lower="${-0.872665 - finger_joint_offset}" upper="${0.872665 - finger_joint_offset}" velocity="2.0" effort="1000" />
       <mimic joint="${prefix}finger_joint" multiplier="1" offset="0" />
     </joint>
@@ -30,5 +38,11 @@
   </xacro:macro>
   <xacro:macro name="finger_joint" params="prefix">
-    <link name="${prefix}finger_width_mock_link"/>
+    <!-- tiny inertia: without it the URDF->SDF conversion drops this link and finger_width with it -->
+    <link name="${prefix}finger_width_mock_link">
+      <inertial>
+        <mass value="0.001" />
+        <inertia ixx="1e-7" ixy="0" ixz="0" iyy="1e-7" iyz="0" izz="1e-7" />
+      </inertial>
+    </link>
     <joint name="${prefix}finger_width" type="prismatic">
       <origin xyz="0 0 0" rpy="0 0 0" />
@@ -39,10 +53,10 @@
     </joint>
     <joint name="${prefix}finger_joint" type="revolute">
-      <origin xyz="0 -0.024112 0.136813" rpy="0 0 0" />
+      <origin xyz="0 -0.024112 0.136813" rpy="${-finger_joint_offset} 0 0" />
       <parent link="${prefix}onrobot_base_link" />
       <child link="${prefix}left_outer_knuckle" />
       <axis xyz="-1 0 0" />
-      <limit lower="-0.628319" upper="0.628319" velocity="2.0" effort="1000" />
-      <mimic joint="${prefix}finger_width" multiplier="${0.88 * ((-0.628319 - 0.628319) / 0.160)}" offset="0.628319" />
+      <limit lower="${-0.628319 - finger_joint_offset}" upper="${0.628319 - finger_joint_offset}" velocity="2.0" effort="1000" />
+      <mimic joint="${prefix}finger_width" multiplier="${finger_joint_multiplier}" offset="0" />
     </joint>
     <xacro:finger_joints prefix="${prefix}" fingerprefix="left" reflect="1.0"/>
@@ -50,9 +64,9 @@
   <xacro:macro name="right_outer_knuckle_joint" params="prefix">
     <joint name="${prefix}right_outer_knuckle_joint" type="revolute">
-      <origin xyz="0 0.024112 0.136813" rpy="0 0 ${pi}" />
+      <origin xyz="0 0.024112 0.136813" rpy="${-finger_joint_offset} 0 ${pi}" />
       <parent link="${prefix}onrobot_base_link" />
       <child link="${prefix}right_outer_knuckle" />
       <axis xyz="1 0 0" />
-      <limit lower="-0.628319" upper="0.628319" velocity="2.0" effort="1000" />
+      <limit lower="${-0.628319 + finger_joint_offset}" upper="${0.628319 + finger_joint_offset}" velocity="2.0" effort="1000" />
       <mimic joint="${prefix}finger_joint" multiplier="-1" offset="0" />
     </joint>

Commit message: feat(rg_macros): add actuated_joint option and closing-side limit slack for gazebo
Co-Authored-By: Claude Opus 5 <noreply@anthropic.com>

File: urdf/rg2_macro.xacro (robot description, xacro)
@@ -9,4 +9,9 @@
   -->
   <xacro:property name="finger_joint_offset" value="0.785398" />
+  <!-- Fully closed (finger_width = 0) would put finger_joint and the knuckles exactly on a
+       position limit. In Gazebo (DART) a velocity-servoed joint resting on its limit ignores
+       further commands (dartsim/dart#1583) and the gripper gets stuck, so the limits on the
+       closing side get a small slack. finger_width limits still bound the real opening. -->
+  <xacro:property name="closed_limit_slack" value="0.05" />
   <xacro:property name="finger_joint_multiplier" value="${0.85 * ((-0.558505 - 0.785398) / 0.110)}" />
   <xacro:include filename="$(find onrobot_description)/urdf/inc/rg_common.xacro" />
@@ -17,5 +22,5 @@
       <child link="${prefix}${fingerprefix}_inner_knuckle" />
       <axis xyz="1 0 0" />
-      <limit lower="${-0.785398 + finger_joint_offset}" upper="${0.785398 + finger_joint_offset}" velocity="100.0" effort="1000" />
+      <limit lower="${-0.785398 + finger_joint_offset - closed_limit_slack}" upper="${0.785398 + finger_joint_offset}" velocity="100.0" effort="1000" />
       <mimic joint="${prefix}finger_joint" multiplier="-1" offset="0" />
     </joint>
@@ -37,5 +42,5 @@
     </joint>
   </xacro:macro>
-  <xacro:macro name="finger_joint" params="prefix">
+  <xacro:macro name="finger_joint" params="prefix actuated_joint">
     <!-- tiny inertia: without it the URDF->SDF conversion drops this link and finger_width with it -->
     <link name="${prefix}finger_width_mock_link">
@@ -51,4 +56,7 @@
       <axis xyz="0 0 1" />
       <limit lower="0" upper="0.110" velocity="0.127" effort="40" />
+      <xacro:if value="${actuated_joint == 'finger_joint'}">
+        <mimic joint="${prefix}finger_joint" multiplier="${1.0 / finger_joint_multiplier}" offset="0" />
+      </xacro:if>
     </joint>
     <joint name="${prefix}finger_joint" type="revolute">
@@ -57,6 +65,8 @@
       <child link="${prefix}left_outer_knuckle" />
       <axis xyz="-1 0 0" />
-      <limit lower="${-0.558505 - finger_joint_offset}" upper="${0.785398 - finger_joint_offset}" velocity="100.0" effort="1000" />
-      <mimic joint="${prefix}finger_width" multiplier="${finger_joint_multiplier}" offset="0" />
+      <limit lower="${-0.558505 - finger_joint_offset}" upper="${0.785398 - finger_joint_offset + closed_limit_slack}" velocity="100.0" effort="1000" />
+      <xacro:if value="${actuated_joint == 'finger_width'}">
+        <mimic joint="${prefix}finger_width" multiplier="${finger_joint_multiplier}" offset="0" />
+      </xacro:if>
     </joint>
     <xacro:finger_joints prefix="${prefix}" fingerprefix="left" reflect="1.0"/>
@@ -68,16 +78,19 @@
       <child link="${prefix}right_outer_knuckle" />
       <axis xyz="1 0 0" />
-      <limit lower="${-0.785398 + finger_joint_offset}" upper="${0.785398 + finger_joint_offset}" velocity="100.0" effort="1000" />
+      <limit lower="${-0.785398 + finger_joint_offset - closed_limit_slack}" upper="${0.785398 + finger_joint_offset}" velocity="100.0" effort="1000" />
       <mimic joint="${prefix}finger_joint" multiplier="-1" offset="0" />
     </joint>
     <xacro:finger_joints prefix="${prefix}" fingerprefix="right" reflect="-1.0"/>
   </xacro:macro>
-  <xacro:macro name="onrobot_rg2" params="prefix">
+  <!-- actuated_joint: finger_width (prismatic opening [m], default, matches the real driver) or
+       finger_joint (knuckle angle [rad], used in Gazebo: driving the massless finger_width
+       slider through the physics engine is unreliable). The other one becomes a mimic. -->
+  <xacro:macro name="onrobot_rg2" params="prefix actuated_joint:=finger_width">
     <xacro:onrobot_base_link prefix="${prefix}" />
     <xacro:finger_links prefix="${prefix}" fingerprefix="left"/>
     <xacro:finger_links prefix="${prefix}" fingerprefix="right"/>
-    <xacro:finger_joint prefix="${prefix}"/>
+    <xacro:finger_joint prefix="${prefix}" actuated_joint="${actuated_joint}"/>
     <xacro:right_outer_knuckle_joint prefix="${prefix}"/>
-    <xacro:transmission_macro prefix="${prefix}" joint_name="finger_width"/>
+    <xacro:transmission_macro prefix="${prefix}" joint_name="${actuated_joint}"/>
     <link name="${prefix}gripper_tcp" />
     <joint name="${prefix}tcp_joint" type="fixed">

File: urdf/rg6_macro.xacro (robot description, xacro)
@@ -9,4 +9,9 @@
   -->
   <xacro:property name="finger_joint_offset" value="0.628319" />
+  <!-- Fully closed (finger_width = 0) would put finger_joint and the knuckles exactly on a
+       position limit. In Gazebo (DART) a velocity-servoed joint resting on its limit ignores
+       further commands (dartsim/dart#1583) and the gripper gets stuck, so the limits on the
+       closing side get a small slack. finger_width limits still bound the real opening. -->
+  <xacro:property name="closed_limit_slack" value="0.05" />
   <xacro:property name="finger_joint_multiplier" value="${0.88 * ((-0.628319 - 0.628319) / 0.160)}" />
   <xacro:include filename="$(find onrobot_description)/urdf/inc/rg_common.xacro" />
@@ -17,5 +22,5 @@
       <child link="${prefix}${fingerprefix}_inner_knuckle" />
       <axis xyz="1 0 0" />
-      <limit lower="${-0.628319 + finger_joint_offset}" upper="${0.628319 + finger_joint_offset}" velocity="2.0" effort="1000" />
+      <limit lower="${-0.628319 + finger_joint_offset - closed_limit_slack}" upper="${0.628319 + finger_joint_offset}" velocity="2.0" effort="1000" />
       <mimic joint="${prefix}finger_joint" multiplier="-1" offset="0" />
     </joint>
@@ -37,5 +42,5 @@
     </joint>
   </xacro:macro>
-  <xacro:macro name="finger_joint" params="prefix">
+  <xacro:macro name="finger_joint" params="prefix actuated_joint">
     <!-- tiny inertia: without it the URDF->SDF conversion drops this link and finger_width with it -->
     <link name="${prefix}finger_width_mock_link">
@@ -51,4 +56,7 @@
       <axis xyz="0 0 1" />
       <limit lower="0" upper="0.160" velocity="0.160" effort="120" />
+      <xacro:if value="${actuated_joint == 'finger_joint'}">
+        <mimic joint="${prefix}finger_joint" multiplier="${1.0 / finger_joint_multiplier}" offset="0" />
+      </xacro:if>
     </joint>
     <joint name="${prefix}finger_joint" type="revolute">
@@ -57,6 +65,8 @@
       <child link="${prefix}left_outer_knuckle" />
       <axis xyz="-1 0 0" />
-      <limit lower="${-0.628319 - finger_joint_offset}" upper="${0.628319 - finger_joint_offset}" velocity="2.0" effort="1000" />
-      <mimic joint="${prefix}finger_width" multiplier="${finger_joint_multiplier}" offset="0" />
+      <limit lower="${-0.628319 - finger_joint_offset}" upper="${0.628319 - finger_joint_offset + closed_limit_slack}" velocity="2.0" effort="1000" />
+      <xacro:if value="${actuated_joint == 'finger_width'}">
+        <mimic joint="${prefix}finger_width" multiplier="${finger_joint_multiplier}" offset="0" />
+      </xacro:if>
     </joint>
     <xacro:finger_joints prefix="${prefix}" fingerprefix="left" reflect="1.0"/>
@@ -68,16 +78,19 @@
       <child link="${prefix}right_outer_knuckle" />
       <axis xyz="1 0 0" />
-      <limit lower="${-0.628319 + finger_joint_offset}" upper="${0.628319 + finger_joint_offset}" velocity="2.0" effort="1000" />
+      <limit lower="${-0.628319 + finger_joint_offset - closed_limit_slack}" upper="${0.628319 + finger_joint_offset}" velocity="2.0" effort="1000" />
       <mimic joint="${prefix}finger_joint" multiplier="-1" offset="0" />
     </joint>
     <xacro:finger_joints prefix="${prefix}" fingerprefix="right" reflect="-1.0"/>
   </xacro:macro>
-  <xacro:macro name="onrobot_rg6" params="prefix">
+  <!-- actuated_joint: finger_width (prismatic opening [m], default, matches the real driver) or
+       finger_joint (knuckle angle [rad], used in Gazebo: driving the massless finger_width
+       slider through the physics engine is unreliable). The other one becomes a mimic. -->
+  <xacro:macro name="onrobot_rg6" params="prefix actuated_joint:=finger_width">
     <xacro:onrobot_base_link prefix="${prefix}" />
     <xacro:finger_links prefix="${prefix}" fingerprefix="left"/>
     <xacro:finger_links prefix="${prefix}" fingerprefix="right"/>
-    <xacro:finger_joint prefix="${prefix}"/>
+    <xacro:finger_joint prefix="${prefix}" actuated_joint="${actuated_joint}"/>
     <xacro:right_outer_knuckle_joint prefix="${prefix}"/>
-    <xacro:transmission_macro prefix="${prefix}" joint_name="finger_width"/>
+    <xacro:transmission_macro prefix="${prefix}" joint_name="${actuated_joint}"/>
     <link name="${prefix}gripper_tcp"/>
     <joint name="${prefix}tcp_joint" type="fixed">
